Commit message: the robot model is ok

File: config/gazebo_custom_env.urdf (robot description, URDF)
Before this commit: robot custom_env, 15 links, 14 joints
Joints:
- removed joint gripper_joint
- added joint enclosure_joint: type fixed, parent tool0, child enclosure, origin xyz=0 0 0 rpy=0 0 0

Commit message: added mesh object

File: config/gazebo_custom_env.urdf (robot description, URDF)
Before this commit: robot custom_env, 15 links, 14 joints
Joints:
- joint robot_base_to_robot_joint: origin xyz=0 0 0 rpy=0 0 1.5707963267948966 -> xyz=0 0 0 rpy=0 0 0
